Commit message: Learning URDF
Made simple URDF file for square car

File: src/robot/description/robot_core.xacro (robot description, xacro)
@@ -1,12 +1,19 @@
 <?xml version="1.0"?>
 <robot xmlns:xacro="http://www.ros.org/wiki/xacro">
+    <xacro:include filename="inertial_macros.xacro"/>
     <!-- Colour options for robot -->
     <material name="blue">
-        <color rgba="0.2 0.2 1 1"/>
+        <color rgba="0.2 1 1 1"/>
+    </material>
+    <material name="black">
+        <color rgba="0 0 0 1"/>
+    </material>
+    <material name="white">
+        <color rgba="1 1 1 1"/>
     </material>
     <!-- Base link is centre of the 2 drive wheels -->
     <link name="base_link">
     </link>
-    <!-- Chassis - box shape with origin just behind the wheels -->
+    <!-- Chassis link - box shape with origin just behind the wheels -->
     <joint name="chassis_joint" type="fixed">
         <parent link="base_link"/>
@@ -18,8 +25,117 @@
             <origin xyz="0.15 0 0.075"/>
             <geometry>
-                <box size"0.3 0.3 0.15"/>
+                <box size="0.4 0.4 0.15"/>
             </geometry>
             <material name="blue"/>
         </visual>
+        <collision>
+            <origin xyz="0.15 0 0.075"/>
+            <geometry>
+                <box size="0.4 0.4 0.15"/>
+            </geometry>
+        </collision>
+        <xacro:inertial_box mass="0.5" x="0.3" y="0.3" z="0.15">
+            <origin xyz="0.15 0 0.075" rpy="0 0 0"/>
+        </xacro:inertial_box>
+    </link>
+    <!-- Left front wheel link -->
+    <joint name="left_front_wheel_joint" type="continuous">
+        <parent link="base_link" />
+        <child link="left_front_wheel"/>
+        <origin xyz="0.175 0.175 0" rpy="-${pi/2} 0 0"/>
+        <axis xyz="0 0 1"/>
+    </joint>
+    <link name="left_front_wheel">
+        <visual>
+            <origin xyz="0 0 0.0"/>
+            <geometry>
+                <cylinder radius="0.05" length="0.04"/>
+            </geometry>
+            <material name="black"/>
+        </visual>
+        <collision>
+            <origin xyz="0 0 0.0"/>v
+            <geometry>
+                <cylinder radius="0.05" length="0.04"/>
+            </geometry>
+        </collision>
+        <xacro:inertial_cylinder mass="0.1" length="0.04" radius="0.05">
+            <origin xyz="0 0 0" rpy="0 0 0"/>
+        </xacro:inertial_cylinder>
+    </link>
+    <!-- Left back wheel link -->
+    <joint name="left_back_wheel_joint" type="continuous">
+        <parent link="base_link" />
+        <child link="left_back_wheel"/>
+        <origin xyz="-0.175 0.175 0" rpy="-${pi/2} 0 0"/>
+        <axis xyz="0 0 1"/>
+    </joint>
+    <link name="left_back_wheel">
+        <visual>
+            <origin xyz="0 0 0.0"/>
+            <geometry>
+                <cylinder radius="0.05" length="0.04"/>
+            </geometry>
+            <material name="black"/>
+        </visual>
+        <collision>
+            <origin xyz="0 0 0.0"/>
+            <geometry>
+                <cylinder radius="0.05" length="0.04"/>
+            </geometry>
+        </collision>
+        <xacro:inertial_cylinder mass="0.1" length="0.04" radius="0.05">
+            <origin xyz="0 0 0" rpy="0 0 0"/>
+        </xacro:inertial_cylinder>
+    </link>
+     <!-- Right front wheel link -->
+    <joint name="right_front_wheel_joint" type="continuous">
+        <parent link="base_link" />
+        <child link="right_front_wheel"/>
+        <origin xyz="0.175 -0.175 0" rpy="${pi/2} 0 0"/>
+        <axis xyz="0 0 -1"/>
+    </joint>
+    <link name="right_front_wheel">
+        <visual>
+            <origin xyz="0 0 0.0"/>
+            <geometry>
+                <cylinder radius="0.05" length="0.04"/>
+            </geometry>
+            <material name="black"/>
+        </visual>
+        <collision>
+            <origin xyz="0 0 0.0"/>
+            <geometry>
+                <cylinder radius="0.05" length="0.04"/>
+            </geometry>
+        </collision>
+        <xacro:inertial_cylinder mass="0.1" length="0.04" radius="0.05">
+            <origin xyz="0 0 0" rpy="0 0 0"/>
+        </xacro:inertial_cylinder>
+    </link>
+     <!-- Right back wheel link -->
+    <joint name="right_back_wheel_joint" type="continuous">
+        <parent link="base_link" />
+        <child link="right_back_wheel"/>
+        <origin xyz="-0.175 -0.175 0" rpy="${pi/2} 0 0"/>
+        <axis xyz="0 0 -1"/>
+    </joint>
+    <link name="right_back_wheel">
+        <visual>
+            <origin xyz="0 0 0.0"/>
+            <geometry>
+                <cylinder radius="0.05" length="0.04"/>
+            </geometry>
+            <material name="black"/>
+        </visual>
+        <collision>
+            <origin xyz="0 0 0.0"/>
+            <geometry>
+                <cylinder radius="0.05" length="0.04"/>
+            </geometry>
+        </collision>
+        <xacro:inertial_cylinder mass="0.1" length="0.04" radius="0.05">
+            <origin xyz="0 0 0" rpy="0 0 0"/>
+        </xacro:inertial_cylinder>
     </link>
 </robot>

Commit message: FS Chassis - WIP

File: src/robot/description/robot_core.xacro (robot description, xacro)
@@ -12,4 +12,7 @@
         <color rgba="1 1 1 1"/>
     </material>
+    <material name="silver">
+        <color rgba="0.430 0.417 0.417 1"/>
+    </material>
     <!-- Base link is centre of the 2 drive wheels -->
     <link name="base_link">
@@ -19,22 +22,22 @@
         <parent link="base_link"/>
         <child link="chassis"/>
-        <origin xyz="-0.1 0 0"/>
+        <origin xyz="-0.4765 0 0"/>
     </joint>
     <link name="chassis">
         <visual>
-            <origin xyz="0.15 0 0.075"/>
+            <origin xyz="0.4765 0 0"/>
             <geometry>
-                <box size="0.4 0.4 0.15"/>
+                <box size="0.953 0.22 0.2"/>
             </geometry>
-            <material name="blue"/>
+            <material name="silver"/>
         </visual>
         <collision>
-            <origin xyz="0.15 0 0.075"/>
+            <origin xyz="0.4765 0 0"/>
             <geometry>
-                <box size="0.4 0.4 0.15"/>
+                <box size="0.953 0.22 0.2"/>
             </geometry>
         </collision>
         <xacro:inertial_box mass="0.5" x="0.3" y="0.3" z="0.15">
-            <origin xyz="0.15 0 0.075" rpy="0 0 0"/>
+            <origin xyz="0.4765 0 0" rpy="0 0 0"/>
         </xacro:inertial_box>
     </link>

Commit message: Updated car urdf file

File: src/robot/description/robot_core.xacro (robot description, xacro)
@@ -4,64 +4,66 @@
     <!-- Colour options for robot -->
     <material name="blue">
-        <color rgba="0.2 1 1 1"/>
+        <color rgba="0.2 0.2 1.0 1.0"/>
     </material>
     <material name="black">
-        <color rgba="0 0 0 1"/>
+        <color rgba="0.0 0.0 0.0 1.0"/>
     </material>
     <material name="white">
-        <color rgba="1 1 1 1"/>
+        <color rgba="1.0 1.0 1.0 1.0"/>
     </material>
     <material name="silver">
-        <color rgba="0.430 0.417 0.417 1"/>
+        <!--color rgba="0.62 0.62 0.62 0.5"/-->
+        <color rgba="0.78 0.72 0.72 1.0"/>
     </material>
     <!-- Base link is centre of the 2 drive wheels -->
     <link name="base_link">
     </link>
-    <!-- Chassis link - box shape with origin just behind the wheels -->
+    <!-- Chassis link - box shape with origin just behind the wheels (l/w/h 964.3/231.23/200)
     <joint name="chassis_joint" type="fixed">
         <parent link="base_link"/>
         <child link="chassis"/>
-        <origin xyz="-0.4765 0 0"/>
+        <origin xyz="0 0 0.12725"/>
     </joint>
     <link name="chassis">
         <visual>
-            <origin xyz="0.4765 0 0"/>
-            <geometry>
-                <box size="0.953 0.22 0.2"/>
-            </geometry>
-            <material name="silver"/>
-        </visual>
-        <collision>
-            <origin xyz="0.4765 0 0"/>
-            <geometry>
-                <box size="0.953 0.22 0.2"/>
+            <origin xyz="0 0 0"/>
+            <geometry>
+                <box size="0.96423 0.22 0.2"/>
+            </geometry>
+            <material name="blue"/>
+        </visual>
+        <collision>
+            <origin xyz="0 0 0"/>
+            <geometry>
+                <box size="0.96423 0.22 0.2"/>
             </geometry>
         </collision>
         <xacro:inertial_box mass="0.5" x="0.3" y="0.3" z="0.15">
-            <origin xyz="0.4765 0 0" rpy="0 0 0"/>
+            <origin xyz="0 0 0" rpy="0 0 0"/>
         </xacro:inertial_box>
     </link>
+    -->
     <!-- Left front wheel link -->
     <joint name="left_front_wheel_joint" type="continuous">
         <parent link="base_link" />
         <child link="left_front_wheel"/>
-        <origin xyz="0.175 0.175 0" rpy="-${pi/2} 0 0"/>
-        <axis xyz="0 0 1"/>
+        <origin xyz="-0.34264 -0.309055 0.12725" rpy="-${pi/2} 0 0"/>
+        <axis xyz="-0.34264 -0.309055 0.12725"/>
     </joint>
     <link name="left_front_wheel">
         <visual>
-            <origin xyz="0 0 0.0"/>
-            <geometry>
-                <cylinder radius="0.05" length="0.04"/>
+            <origin xyz="0 0 0"/>
+            <geometry>
+                <cylinder radius="0.12725" length="0.1144"/>
             </geometry>
             <material name="black"/>
         </visual>
         <collision>
-            <origin xyz="0 0 0.0"/>v
-            <geometry>
-                <cylinder radius="0.05" length="0.04"/>
-            </geometry>
-        </collision>
-        <xacro:inertial_cylinder mass="0.1" length="0.04" radius="0.05">
+            <origin xyz="0 0 0"/>v
+            <geometry>
+                <cylinder radius="0.12725" length="0.1144"/>
+            </geometry>
+        </collision>
+        <xacro:inertial_cylinder mass="0.1" length="0.1144" radius="0.12725">
             <origin xyz="0 0 0" rpy="0 0 0"/>
         </xacro:inertial_cylinder>
@@ -71,22 +73,22 @@
         <parent link="base_link" />
         <child link="left_back_wheel"/>
-        <origin xyz="-0.175 0.175 0" rpy="-${pi/2} 0 0"/>
-        <axis xyz="0 0 1"/>
+        <origin xyz="0.34264 -0.309055 0.12725" rpy="-${pi/2} 0 0"/>
+        <axis xyz="0.34264 -0.309055 0.12725"/>
     </joint>
     <link name="left_back_wheel">
         <visual>
-            <origin xyz="0 0 0.0"/>
-            <geometry>
-                <cylinder radius="0.05" length="0.04"/>
+            <origin xyz="0 0 0"/>
+            <geometry>
+                <cylinder radius="0.12725" length="0.1144"/>
             </geometry>
             <material name="black"/>
         </visual>
         <collision>
-            <origin xyz="0 0 0.0"/>
-            <geometry>
-                <cylinder radius="0.05" length="0.04"/>
-            </geometry>
-        </collision>
-        <xacro:inertial_cylinder mass="0.1" length="0.04" radius="0.05">
+            <origin xyz="0 0 0"/>
+            <geometry>
+                <cylinder radius="0.12725" length="0.1144"/>
+            </geometry>
+        </collision>
+        <xacro:inertial_cylinder mass="0.1" length="0.1144" radius="0.12725">
             <origin xyz="0 0 0" rpy="0 0 0"/>
         </xacro:inertial_cylinder>
@@ -96,22 +98,22 @@
         <parent link="base_link" />
         <child link="right_front_wheel"/>
-        <origin xyz="0.175 -0.175 0" rpy="${pi/2} 0 0"/>
-        <axis xyz="0 0 -1"/>
+        <origin xyz="-0.34264 0.309055 0.12725" rpy="${pi/2} 0 0"/>
+        <axis xyz="-0.34264 0.309055 0.12725"/>
     </joint>
     <link name="right_front_wheel">
         <visual>
-            <origin xyz="0 0 0.0"/>
-            <geometry>
-                <cylinder radius="0.05" length="0.04"/>
+            <origin xyz="0 0 0"/>
+            <geometry>
+                <cylinder radius="0.12725" length="0.1144"/>
             </geometry>
             <material name="black"/>
         </visual>
         <collision>
-            <origin xyz="0 0 0.0"/>
-            <geometry>
-                <cylinder radius="0.05" length="0.04"/>
-            </geometry>
-        </collision>
-        <xacro:inertial_cylinder mass="0.1" length="0.04" radius="0.05">
+            <origin xyz="0 0 0"/>
+            <geometry>
+                <cylinder radius="0.12725" length="0.1144"/>
+            </geometry>
+        </collision>
+        <xacro:inertial_cylinder mass="0.1" length="0.1144" radius="0.12725">
             <origin xyz="0 0 0" rpy="0 0 0"/>
         </xacro:inertial_cylinder>
@@ -121,22 +123,672 @@
         <parent link="base_link" />
         <child link="right_back_wheel"/>
-        <origin xyz="-0.175 -0.175 0" rpy="${pi/2} 0 0"/>
-        <axis xyz="0 0 -1"/>
+        <origin xyz="0.34264 0.309055 0.12725" rpy="${pi/2} 0 0"/>
+        <axis xyz="0.34264 0.309055 0.12725"/>
     </joint>
     <link name="right_back_wheel">
         <visual>
-            <origin xyz="0 0 0.0"/>
-            <geometry>
-                <cylinder radius="0.05" length="0.04"/>
+            <origin xyz="0 0 0"/>
+            <geometry>
+                <cylinder radius="0.12725" length="0.1144"/>
             </geometry>
             <material name="black"/>
         </visual>
         <collision>
-            <origin xyz="0 0 0.0"/>
-            <geometry>
-                <cylinder radius="0.05" length="0.04"/>
-            </geometry>
-        </collision>
-        <xacro:inertial_cylinder mass="0.1" length="0.04" radius="0.05">
+            <origin xyz="0 0 0"/>
+            <geometry>
+                <cylinder radius="0.12725" length="0.1144"/>
+            </geometry>
+        </collision>
+        <xacro:inertial_cylinder mass="0.1" length="0.1144" radius="0.12725">
+            <origin xyz="0 0 0" rpy="0 0 0"/>
+        </xacro:inertial_cylinder>
+    </link>
+    <!-- Left front suspension -->
+    <joint name="left_front_suspension_joint" type="continuous">
+        <parent link="base_link"/>
+        <child link="left_front_suspension"/>
+        <origin xyz="-0.34264 -0.183735 0.12725" rpy="${pi/2} 0 0"/>
+        <axis xyz="-0.34264 -0.183735 0.12725"/>
+    </joint>
+    <link name="left_front_suspension">
+        <visual>
+            <origin xyz="0 0 0"/>
+            <geometry>
+                <cylinder radius="0.0225" length="0.13624"/>
+            </geometry>
+            <material name="white"/>
+        </visual>
+        <collision>
+            <origin xyz="0 0 0"/>
+            <geometry>
+                <cylinder radius="0.0225" length="0.13624"/>
+            </geometry>
+        </collision>
+        <xacro:inertial_cylinder mass="0.1" length="0.13624" radius="0.0225">
+            <origin xyz="0 0 0" rpy="0 0 0"/>
+        </xacro:inertial_cylinder>
+    </link>
+    <!-- Left back suspension -->
+    <joint name="left_back_suspension_joint" type="continuous">
+        <parent link="base_link"/>
+        <child link="left_back_suspension"/>
+        <origin xyz="0.34264 -0.183735 0.12725" rpy="${pi/2} 0 0"/>
+        <axis xyz="0.34264 -0.183735 0.12725"/>
+    </joint>
+    <link name="left_back_suspension">
+        <visual>
+            <origin xyz="0 0 0"/>
+            <geometry>
+                <cylinder radius="0.0225" length="0.13624"/>
+            </geometry>
+            <material name="white"/>
+        </visual>
+        <collision>
+            <origin xyz="0 0 0"/>
+            <geometry>
+                <cylinder radius="0.0255" length="0.13624"/>
+            </geometry>
+        </collision>
+        <xacro:inertial_cylinder mass="0.1" length="0.13624" radius="0.0225">
+            <origin xyz="0 0 0" rpy="0 0 0"/>
+        </xacro:inertial_cylinder>
+    </link>
+    <!-- Right front suspension -->
+    <joint name="right_front_suspension_joint" type="continuous">
+        <parent link="base_link"/>
+        <child link="right_front_suspension"/>
+        <origin xyz="-0.34264 0.183735 0.12725" rpy="${pi/2} 0 0"/>
+        <axis xyz="-0.34264 0.183735 0.12725"/>
+    </joint>
+    <link name="right_front_suspension">
+        <visual>
+            <origin xyz="0 0 0"/>
+            <geometry>
+                <cylinder radius="0.0225" length="0.13624"/>
+            </geometry>
+            <material name="white"/>
+        </visual>
+        <collision>
+            <origin xyz="0 0 0"/>
+            <geometry>
+                <cylinder radius="0.0225" length="0.13624"/>
+            </geometry>
+        </collision>
+        <xacro:inertial_cylinder mass="0.1" length="0.13624" radius="0.0255">
+            <origin xyz="0 0 0" rpy="0 0 0"/>
+        </xacro:inertial_cylinder>
+    </link>
+    <!-- Right back suspension -->
+    <joint name="right_back_suspension_joint" type="continuous">
+        <parent link="base_link"/>
+        <child link="right_back_suspension"/>
+        <origin xyz="0.34264 0.183735 0.12725" rpy="${pi/2} 0 0"/>
+        <axis xyz="0.34264 0.183735 0.12725"/>
+    </joint>
+    <link name="right_back_suspension">
+        <visual>
+            <origin xyz="0 0 0"/>
+            <geometry>
+                <cylinder radius="0.0225" length="0.13624"/>
+            </geometry>
+            <material name="white"/>
+        </visual>
+        <collision>
+            <origin xyz="0 0 0"/>
+            <geometry>
+                <cylinder radius="0.0225" length="0.13624"/>
+            </geometry>
+        </collision>
+        <xacro:inertial_cylinder mass="0.1" length="0.13624" radius="0.0225">
+            <origin xyz="0 0 0" rpy="0 0 0"/>
+        </xacro:inertial_cylinder>
+    </link>
+    <!-- Chassis pole top right (l/d 964.3/15.88)-->
+    <joint name="chassis_pole_tr_joint" type="fixed">
+        <parent link="base_link"/>
+        <child link="chassis_pole_tr"/>
+        <origin xyz="0 0.115615 0.26225" rpy="0 ${pi/2} 0"/>
+        <axis xyz="0 0.115615 0.26225"/>
+    </joint>
+    <link name="chassis_pole_tr">
+        <visual>
+            <origin xyz="0 0 0"/>
+            <geometry>
+                <cylinder radius="0.01588" length="0.9643"/>
+            </geometry>
+            <material name="silver"/>
+        </visual>
+        <collision>
+            <origin xyz="0 0 0"/>
+            <geometry>
+                <cylinder radius="0.01588" length="0.9643"/>
+            </geometry>
+        </collision>
+        <xacro:inertial_cylinder mass="0.1" length="0.9643" radius="0.01588">
+            <origin xyz="0 0 0" rpy="0 0 0"/>
+        </xacro:inertial_cylinder>
+    </link>
+    <!-- Chassis pole bottom right -->
+    <joint name="chassis_pole_br_joint" type="fixed">
+        <parent link="base_link"/>
+        <child link="chassis_pole_br"/>
+        <origin xyz="0 0.115615 0.06225" rpy="0 ${pi/2} 0"/>
+        <axis xyz="0 0.115615 0.06225"/>
+    </joint>
+    <link name="chassis_pole_br">
+        <visual>
+            <origin xyz="0 0 0"/>
+            <geometry>
+                <cylinder radius="0.01588" length="00.9643"/>
+            </geometry>
+            <material name="silver"/>
+        </visual>
+        <collision>
+            <origin xyz="0 0 0"/>
+            <geometry>
+                <cylinder radius="0.01588" length="0.9643"/>
+            </geometry>
+        </collision>
+        <xacro:inertial_cylinder mass="0.1" length="0.9643" radius="0.01588">
+            <origin xyz="0 0 0" rpy="0 0 0"/>
+        </xacro:inertial_cylinder>
+    </link>
+    <!-- Chassis pole top left -->
+    <joint name="chassis_pole_tl_joint" type="fixed">
+        <parent link="base_link"/>
+        <child link="chassis_pole_tl"/>
+        <origin xyz="0 -0.115615 0.26225" rpy="0 ${pi/2} 0"/>
+        <axis xyz="0 -0.115615 0.26225"/>
+    </joint>
+    <link name="chassis_pole_tl">
+        <visual>
+            <origin xyz="0 0 0"/>
+            <geometry>
+                <cylinder radius="0.01588" length="0.9643"/>
+            </geometry>
+            <material name="silver"/>
+        </visual>
+        <collision>
+            <origin xyz="0 0 0"/>
+            <geometry>
+                <cylinder radius="0.01588" length="0.9643"/>
+            </geometry>
+        </collision>
+        <xacro:inertial_cylinder mass="0.1" length="0.9643" radius="0.01588">
+            <origin xyz="0 0 0" rpy="0 0 0"/>
+        </xacro:inertial_cylinder>
+    </link>
+    <!-- Chassis pole bottom left -->
+    <joint name="chassis_pole_bl_joint" type="fixed">
+        <parent link="base_link"/>
+        <child link="chassis_pole_bl"/>
+        <origin xyz="0 -0.115615 0.06225" rpy="0 ${pi/2} 0"/>
+        <axis xyz="0 -0.115615 0.06225"/>
+    </joint>
+    <link name="chassis_pole_bl">
+        <visual>
+            <origin xyz="0 0 0"/>
+            <geometry>
+                <cylinder radius="0.01588" length="0.9643"/>
+            </geometry>
+            <material name="silver"/>
+        </visual>
+        <collision>
+            <origin xyz="0 0 0"/>
+            <geometry>
+                <cylinder radius="0.01588" length="0.9643"/>
+            </geometry>
+        </collision>
+        <xacro:inertial_cylinder mass="0.1" length="0.9643" radius="0.01588">
+            <origin xyz="0 0 0" rpy="0 0 0"/>
+        </xacro:inertial_cylinder>
+    </link>
+    <!-- Chassis pole bottom front -->
+    <joint name="chassis_pole_bf_joint" type="fixed">
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