Commit message: Adding Gazebo Controls

File: src/robot/description/robot_core.xacro (robot description, xacro)
@@ -69,4 +69,8 @@
         </xacro:inertial_cylinder>
     </link>
+    <!-- To show colour on gazebo -->
+    <gazebo reference="left_front_wheel">
+        <material>Gazebo/Black</material>
+    </gazebo>
     <!-- Left back wheel link -->
     <joint name="left_back_wheel_joint" type="continuous">
@@ -94,4 +98,7 @@
         </xacro:inertial_cylinder>
     </link>
+    <gazebo reference="left_back_wheel">
+        <material>Gazebo/Black</material>
+    </gazebo>
      <!-- Right front wheel link -->
     <joint name="right_front_wheel_joint" type="continuous">
@@ -119,4 +126,7 @@
         </xacro:inertial_cylinder>
     </link>
+    <gazebo reference="right_front_wheel">
+        <material>Gazebo/Black</material>
+    </gazebo>
      <!-- Right back wheel link -->
     <joint name="right_back_wheel_joint" type="continuous">
@@ -144,4 +154,7 @@
         </xacro:inertial_cylinder>
     </link>
+    <gazebo reference="right_back_wheel">
+        <material>Gazebo/Black</material>
+    </gazebo>
     <!-- Left front suspension -->
     <joint name="left_front_suspension_joint" type="continuous">
@@ -169,4 +182,7 @@
         </xacro:inertial_cylinder>
     </link>
+    <gazebo reference="left_front_suspension">
+        <material>Gazebo/White</material>
+    </gazebo>
     <!-- Left back suspension -->
     <joint name="left_back_suspension_joint" type="continuous">
@@ -194,4 +210,7 @@
         </xacro:inertial_cylinder>
     </link>
+    <gazebo reference="left_back_suspension">
+        <material>Gazebo/White</material>
+    </gazebo>
     <!-- Right front suspension -->
     <joint name="right_front_suspension_joint" type="continuous">
@@ -219,4 +238,7 @@
         </xacro:inertial_cylinder>
     </link>
+    <gazebo reference="right_front_suspension">
+        <material>Gazebo/White</material>
+    </gazebo>
     <!-- Right back suspension -->
     <joint name="right_back_suspension_joint" type="continuous">
@@ -244,4 +266,7 @@
         </xacro:inertial_cylinder>
     </link>
+    <gazebo reference="right_back_suspension">
+        <material>Gazebo/White</material>
+    </gazebo>
     <!-- Chassis pole top right (l/d 964.3/15.88)-->
     <joint name="chassis_pole_tr_joint" type="fixed">
@@ -269,4 +294,7 @@
         </xacro:inertial_cylinder>
     </link>
+    <gazebo reference="chassis_pole_tr">
+        <material>Gazebo/Silver</material>
+    </gazebo>
     <!-- Chassis pole bottom right -->
     <joint name="chassis_pole_br_joint" type="fixed">
@@ -294,4 +322,7 @@
         </xacro:inertial_cylinder>
     </link>
+    <gazebo reference="chassis_pole_br">
+        <material>Gazebo/Silver</material>
+    </gazebo>
     <!-- Chassis pole top left -->
     <joint name="chassis_pole_tl_joint" type="fixed">
@@ -319,4 +350,7 @@
         </xacro:inertial_cylinder>
     </link>
+    <gazebo reference="chassis_pole_tl">
+        <material>Gazebo/Silver</material>
+    </gazebo>
     <!-- Chassis pole bottom left -->
     <joint name="chassis_pole_bl_joint" type="fixed">
@@ -344,4 +378,7 @@
         </xacro:inertial_cylinder>
     </link>
+    <gazebo reference="chassis_pole_bl">
+        <material>Gazebo/Silver</material>
+    </gazebo>
     <!-- Chassis pole bottom front -->
     <joint name="chassis_pole_bf_joint" type="fixed">
@@ -369,4 +406,7 @@
         </xacro:inertial_cylinder>
     </link>
+    <gazebo reference="chassis_pole_bf">
+        <material>Gazebo/Silver</material>
+    </gazebo>
     <!-- Chassis pole top front -->
     <joint name="chassis_pole_tf_joint" type="fixed">
@@ -394,4 +434,7 @@
         </xacro:inertial_cylinder>
     </link>
+    <gazebo reference="chassis_pole_tf">
+        <material>Gazebo/Silver</material>
+    </gazebo>
     <!-- Chassis pole bottom back -->
     <joint name="chassis_pole_bb_joint" type="fixed">
@@ -419,4 +462,7 @@
         </xacro:inertial_cylinder>
     </link>
+    <gazebo reference="chassis_pole_bb">
+        <material>Gazebo/Silver</material>
+    </gazebo>
     <!-- Chassis pole top back -->
     <joint name="chassis_pole_tb_joint" type="fixed">
@@ -444,4 +490,7 @@
         </xacro:inertial_cylinder>
     </link>
+    <gazebo reference="chassis_pole_tb">
+        <material>Gazebo/Silver</material>
+    </gazebo>
     <!-- Chassis pole vertical front left -->
     <joint name="chassis_pole_vfl_joint" type="fixed">
@@ -469,4 +518,7 @@
         </xacro:inertial_cylinder>
     </link>
+    <gazebo reference="chassis_pole_vfl">
+        <material>Gazebo/Silver</material>
+    </gazebo>
     <!-- Chassis pole vertical front right -->
     <joint name="chassis_pole_vfr_joint" type="fixed">
@@ -494,4 +546,7 @@
         </xacro:inertial_cylinder>
     </link>
+    <gazebo reference="chassis_pole_vfr">
+        <material>Gazebo/Silver</material>
+    </gazebo>
     <!-- Chassis pole vertical back left -->
     <joint name="chassis_pole_vbl_joint" type="fixed">
@@ -519,4 +574,7 @@
         </xacro:inertial_cylinder>
     </link>
+    <gazebo reference="chassis_pole_vbl">
+        <material>Gazebo/Silver</material>
+    </gazebo>
     <!-- Chassis pole vertical back right -->
     <joint name="chassis_pole_vbr_joint" type="fixed">
@@ -544,4 +602,7 @@
         </xacro:inertial_cylinder>
     </link>
+    <gazebo reference="chassis_pole_vbr">
+        <material>Gazebo/Silver</material>
+    </gazebo>
     <!-- Chassis pole top back angle -->
     <joint name="chassis_pole_tba_joint" type="fixed">
@@ -569,4 +630,7 @@
         </xacro:inertial_cylinder>
     </link>
+    <gazebo reference="chassis_pole_tba">
+        <material>Gazebo/Silver</material>
+    </gazebo>
     <!-- Chassis pole top front angle >
     <joint name="chassis_pole_tfa_joint" type="fixed">
@@ -593,5 +657,8 @@
             <origin xyz="0 0 0" rpy="0 0 0"/>
         </xacro:inertial_cylinder>
-    </link-->
+    </link>
+    <gazebo reference="chassis_pole_tfa">
+        <material>Gazebo/Silver</material>
+    </gazebo-->
  <!-- Chassis pole top back straight -->
     <joint name="chassis_pole_tbs_joint" type="fixed">
@@ -619,4 +686,7 @@
         </xacro:inertial_cylinder>
     </link>
+    <gazebo reference="chassis_pole_tbs">
+        <material>Gazebo/Silver</material>
+    </gazebo>
     <!-- Chassis pole left back straight -->
     <joint name="chassis_pole_lbs_joint" type="fixed">
@@ -644,4 +714,7 @@
         </xacro:inertial_cylinder>
     </link>
+    <gazebo reference="chassis_pole_lbs">
+        <material>Gazebo/Silver</material>
+    </gazebo>
     <!-- Chassis pole right back straight -->
     <joint name="chassis_pole_rbs_joint" type="fixed">
@@ -669,4 +742,7 @@
         </xacro:inertial_cylinder>
     </link>
+    <gazebo reference="chassis_pole_rbs">
+        <material>Gazebo/Silver</material>
+    </gazebo>
  <!-- Chassis pole top front straight -->
     <joint name="chassis_pole_tfs_joint" type="fixed">
@@ -694,4 +770,7 @@
         </xacro:inertial_cylinder>
     </link>
+    <gazebo reference="chassis_pole_tfs">
+        <material>Gazebo/Silver</material>
+    </gazebo>
     <!-- Chassis pole left front straight -->
     <joint name="chassis_pole_lfs_joint" type="fixed">
@@ -719,4 +798,7 @@
         </xacro:inertial_cylinder>
     </link>
+    <gazebo reference="chassis_pole_lfs">
+        <material>Gazebo/Silver</material>
+    </gazebo>
     <!-- Chassis pole right front straight -->
     <joint name="chassis_pole_rfs_joint" type="fixed">
@@ -744,4 +826,7 @@
         </xacro:inertial_cylinder>
     </link>
+    <gazebo reference="chassis_pole_rfs">
+        <material>Gazebo/Silver</material>
+    </gazebo>
  <!-- Chassis pole bottom cross -->
     <joint name="chassis_pole_bc_joint" type="fixed">
@@ -769,4 +854,7 @@
         </xacro:inertial_cylinder>
     </link>
+    <gazebo reference="chassis_pole_bc">
+        <material>Gazebo/Silver</material>
+    </gazebo>
     <!-- Chassis pole bottom cross cross-->
     <joint name="chassis_pole_bcc_joint" type="fixed">
@@ -794,3 +882,6 @@
         </xacro:inertial_cylinder>
     </link>
+    <gazebo reference="chassis_pole_bcc">
+        <material>Gazebo/Silver</material>
+    </gazebo>
 </robot>
