Commit message: Trying to get car to move

File: src/car_sim/description/robot.urdf.xacro (robot description, xacro)
@@ -2,7 +2,3 @@
 <robot xmlns:xacro="http://www.ros.org/wiki/xacro"  name="robot">
     <xacro:include filename="test.xacro" />
-    <!-- Information for Gazebo controls -->
-    <xacro:include filename="gazebo_control.xacro"/>
-    <!-- Information for Lidar -->
-    <xacro:include filename="lidar.xacro"/>
 </robot>

File: src/car_sim/description/robot_core.xacro (robot description, xacro)
@@ -158,5 +158,5 @@
     </gazebo>
     <!-- Left front suspension -->
-    <joint name="left_front_suspension_joint" type="continuous">
+    <joint name="left_front_suspension_joint" type="fixed">
         <parent link="base_link"/>
         <child link="left_front_suspension"/>
@@ -186,5 +186,5 @@
     </gazebo>
     <!-- Left back suspension -->
-    <joint name="left_back_suspension_joint" type="continuous">
+    <joint name="left_back_suspension_joint" type="fixed">
         <parent link="base_link"/>
         <child link="left_back_suspension"/>
@@ -214,5 +214,5 @@
     </gazebo>
     <!-- Right front suspension -->
-    <joint name="right_front_suspension_joint" type="continuous">
+    <joint name="right_front_suspension_joint" type="fixed">
         <parent link="base_link"/>
         <child link="right_front_suspension"/>
@@ -242,5 +242,5 @@
     </gazebo>
     <!-- Right back suspension -->
-    <joint name="right_back_suspension_joint" type="continuous">
+    <joint name="right_back_suspension_joint" type="fixed">
         <parent link="base_link"/>
         <child link="right_back_suspension"/>

File: src/car_sim/description/test.xacro (robot description, xacro)
@@ -59,5 +59,5 @@
         </visual>
         <collision>
-            <origin xyz="0 0 0"/>v
+            <origin xyz="0 0 0"/>
             <geometry>
                 <cylinder radius="0.12725" length="0.1144"/>
@@ -157,5 +157,5 @@
     </gazebo>
     <!-- Left front suspension -->
-    <joint name="left_front_suspension_joint" type="continuous">
+    <joint name="left_front_suspension_joint" type="fixed">
         <parent link="base_link"/>
         <child link="left_front_suspension"/>
@@ -185,5 +185,5 @@
     </gazebo>
     <!-- Left back suspension -->
-    <joint name="left_back_suspension_joint" type="continuous">
+    <joint name="left_back_suspension_joint" type="fixed">
         <parent link="base_link"/>
         <child link="left_back_suspension"/>
@@ -213,5 +213,5 @@
     </gazebo>
     <!-- Right front suspension -->
-    <joint name="right_front_suspension_joint" type="continuous">
+    <joint name="right_front_suspension_joint" type="fixed">
         <parent link="base_link"/>
         <child link="right_front_suspension"/>
@@ -241,5 +241,5 @@
     </gazebo>
     <!-- Right back suspension -->
-    <joint name="right_back_suspension_joint" type="continuous">
+    <joint name="right_back_suspension_joint" type="fixed">
         <parent link="base_link"/>
         <child link="right_back_suspension"/>
@@ -268,3 +268,52 @@
         <material>Gazebo/White</material>
     </gazebo>
+    <joint name="lidar_joint" type="fixed">
+        <parent link="chassis"/>
+        <child link="lidar_frame"/>
+        <origin xyz="0 0 0.12" rpy="0 0 0"/>
+    </joint>
+    <link name="lidar_frame">
+        <visual>
+            <geometry>
+                <cylinder radius="0.05" length="0.04"/>
+            </geometry>
+            <material name="blue"/>
+        </visual>
+        <collision>
+            <geometry>
+                <cylinder radius="0.05" length="0.04"/>
+            </geometry>
+        </collision>
+        <xacro:inertial_cylinder mass="0.1" length="0.04" radius="0.05">
+            <origin xyz="0 0 0.12" rpy="0 0 0"/>
+        </xacro:inertial_cylinder>
+    </link>
+    <gazebo reference="lidar_frame">
+        <sensor name="lidar" type="gpu_ray">  <!-- ray means its a scanning laser -->
+            <pose> 0 0 0 0 0 0 </pose>  <!-- origin of lidar is at origin of link -->
+            <visualize>true</visualize>
+            <update_rate>10</update_rate> <!-- update laser 10 times a second -->
+            <ray>
+                <scan>
+                    <horizontal> <!-- scanning horizontally with 360 samples a resolution -->
+                        <samples>360</samples>
+                        <resolution>1</resolution>
+                        <min_angle>-3.14</min_angle>  <!-- angle of -180 to 180 degrees in radians -->
+                        <max_angle>3.14</max_angle>
+                    </horizontal>
+                </scan>
+                <range>
+                    <min>0.3</min>
+                    <max>12</max>
+                    <resolution>0.01</resolution>
+                </range>
+            </ray>
+            <plugin name="laser_controller" filename="libgazebo_ros_gpu_laser.so">
+                <topicName>/rrbot/laser/scan</topicName>
+                <frameName>lidar_frame</frameName>
+            </plugin>
+        </sensor>
+    </gazebo>
+    <!-- Motor Simulation -->
+	<xacro:include filename="test.gazebo" />
 </robot>
